File: resources/netclock-wirelayout/SSD-LAYOUT.sch (KiCad schematic (older format))
At the start: 6 parts, among them J1 SSD-SEG, J2 SSD-DATA, U1 FJS23101BH, U2 FJS23101BH, U3 FJS23101BH, U4 FJS23101BH

Commit message: Update 7-segment display details in the wiring layout.
Other:
- note added: "2.3 inch (57 mm) 7.2V single digit - Red."
- note added: "Common anode 7-segment display."
- note added: "Hour Segment 1"
- note added: "Hour Segment 2"
- note added: "Minute Segment 1"
- note added: "Minute Segment 2"
- note added: "U1...U4:"
Changed lines of the file:
@@
 Text Label 8550 2700 0    50   ~ 0
 A3
+Text Notes 2050 5550 0    50   ~ 0
+U1...U4:
+Text Notes 2400 5700 0    50   ~ 0
+2.3 inch (57 mm) 7.2V single digit - Red.
+Text Notes 2400 5550 0    50   ~ 0
+Common anode 7-segment display.
+Text Notes 2850 2750 0    50   ~ 0
+Hour Segment 1
+Text Notes 4450 2750 0    50   ~ 0
+Hour Segment 2
+Text Notes 5950 2750 0    50   ~ 0
+Minute Segment 1
+Text Notes 7550 2750 0    50   ~ 0
+Minute Segment 2
 $EndSCHEMATC
